File: Matrix.sch (KiCad schematic (older format))
At the start: 226 parts

Commit message: Update: Work on bottom row layouts
Parts:
- K_LALT2, K_LCTL2: footprint MX_Alps_Hybrid:MX-1.5U -> MX_Alps_Hybrid:MX-1.5U-FLIPPED
- K_LGUI2, K_RALT3, K_RCTL2, K_RMOD2: footprint MX_Alps_Hybrid:MX-1U -> MX_Alps_Hybrid:MX-1U-FLIPPED
- K_SPACE1_1: footprint MX_Alps_Hybrid:MX-2.25U -> MX_Alps_Hybrid:MX-2.25U-ReversedStabilizers
- K_SPACE1_2: footprint MX_Alps_Hybrid:MX-2.75U -> MX_Alps_Hybrid:MX-2.75U-FLIPPED-ReversedStabilizers
- K_SPACE1_3, K_SPACE3_1, K_SPACE3_3: footprint MX_Alps_Hybrid:MX-2.75U -> MX_Alps_Hybrid:MX-2.75U-ReversedStabilizers
- K_SPACE2_1, K_SPACE2_5: footprint MX_Alps_Hybrid:MX-1.25U -> MX_Alps_Hybrid:MX-1.25U-FLIPPED
- K_SPACE2_2: footprint MX_Alps_Hybrid:MX-6.25U -> MX_Alps_Hybrid:MX-6.25U-ReversedStabilizers
- K_SPACE2_3: footprint MX_Alps_Hybrid:MX-7U -> MX_Alps_Hybrid:MX-7U-ReversedStabilizers
- K_SPACE3_2: footprint MX_Alps_Hybrid:MX-2.25U -> MX_Alps_Hybrid:MX-2.25U-FLIPPED-ReversedStabilizers
Changed lines of the file:
@@
 F 0 "K_LCTL2" H 1550 4580 60  0000 C CNN
 F 1 "MX-1.5U" H 1550 4505 20  0000 C CNN
-F 2 "MX_Alps_Hybrid:MX-1.5U" H 1525 4430 60  0001 C CNN
+F 2 "MX_Alps_Hybrid:MX-1.5U-FLIPPED" H 1525 4430 60  0001 C CNN
 F 3 "" H 1525 4430 60  0001 C CNN
 	1    1550 4455
@@
 F 0 "K_LGUI2" H 2050 4580 60  0000 C CNN
 F 1 "MX-1U" H 2050 4505 20  0000 C CNN
-F 2 "MX_Alps_Hybrid:MX-1U" H 2025 4430 60  0001 C CNN
+F 2 "MX_Alps_Hybrid:MX-1U-FLIPPED" H 2025 4430 60  0001 C CNN
 F 3 "" H 2025 4430 60  0001 C CNN
 	1    2050 4455
@@
 F 0 "K_SPACE1_1" H 3400 3925 60  0000 C CNN
 F 1 "MX-2.25U" H 3400 3850 20  0000 C CNN
-F 2 "MX_Alps_Hybrid:MX-2.25U" H 3375 3775 60  0001 C CNN
+F 2 "MX_Alps_Hybrid:MX-2.25U-ReversedStabilizers" H 3375 3775 60  0001 C CNN
 F 3 "" H 3375 3775 60  0001 C CNN
 	1    3400 3800
@@
 F 0 "K_SPACE2_1" H 4300 3925 60  0000 C CNN
 F 1 "MX-1.25U" H 4300 3850 20  0000 C CNN
-F 2 "MX_Alps_Hybrid:MX-1.25U" H 4275 3775 60  0001 C CNN
+F 2 "MX_Alps_Hybrid:MX-1.25U-FLIPPED" H 4275 3775 60  0001 C CNN
 F 3 "" H 4275 3775 60  0001 C CNN
 	1    4300 3800
@@
 F 0 "K_SPACE3_1" H 5200 3925 60  0000 C CNN
 F 1 "MX-2.75U" H 5200 3850 20  0000 C CNN
-F 2 "MX_Alps_Hybrid:MX-2.75U" H 5175 3775 60  0001 C CNN
+F 2 "MX_Alps_Hybrid:MX-2.75U-ReversedStabilizers" H 5175 3775 60  0001 C CNN
 F 3 "" H 5175 3775 60  0001 C CNN
 	1    5200 3800
@@
 F 0 "K_SPACE1_2" H 3400 4575 60  0000 C CNN
 F 1 "MX-2.75U" H 3400 4500 20  0000 C CNN
-F 2 "MX_Alps_Hybrid:MX-2.75U" H 3375 4425 60  0001 C CNN
+F 2 "MX_Alps_Hybrid:MX-2.75U-FLIPPED-ReversedStabilizers" H 3375 4425 60  0001 C CNN
 F 3 "" H 3375 4425 60  0001 C CNN
 	1    3400 4450
@@
 F 0 "K_SPACE3_2" H 5200 4575 60  0000 C CNN
 F 1 "MX-2.25U" H 5200 4500 20  0000 C CNN
-F 2 "MX_Alps_Hybrid:MX-2.25U" H 5175 4425 60  0001 C CNN
+F 2 "MX_Alps_Hybrid:MX-2.25U-FLIPPED-ReversedStabilizers" H 5175 4425 60  0001 C CNN
 F 3 "" H 5175 4425 60  0001 C CNN
 	1    5200 4450
@@
 F 0 "K_SPACE2_2" H 4300 4575 60  0000 C CNN
 F 1 "MX-6.25U" H 4300 4500 20  0000 C CNN
-F 2 "MX_Alps_Hybrid:MX-6.25U" H 4275 4425 60  0001 C CNN
+F 2 "MX_Alps_Hybrid:MX-6.25U-ReversedStabilizers" H 4275 4425 60  0001 C CNN
 F 3 "" H 4275 4425 60  0001 C CNN
 	1    4300 4450
@@
 F 0 "K_RALT3" H 6100 5075 60  0000 C CNN
 F 1 "MX-1U" H 6100 5000 20  0000 C CNN
-F 2 "MX_Alps_Hybrid:MX-1U" H 6075 4925 60  0001 C CNN
+F 2 "MX_Alps_Hybrid:MX-1U-FLIPPED" H 6075 4925 60  0001 C CNN
 F 3 "" H 6075 4925 60  0001 C CNN
 	1    6100 4950
@@
 F 0 "K_SPACE2_3" H 4300 5095 60  0000 C CNN
 F 1 "MX-7U" H 4300 5020 20  0000 C CNN
-F 2 "MX_Alps_Hybrid:MX-7U" H 4275 4945 60  0001 C CNN
+F 2 "MX_Alps_Hybrid:MX-7U-ReversedStabilizers" H 4275 4945 60  0001 C CNN
 F 3 "" H 4275 4945 60  0001 C CNN
 	1    4300 4970
@@
 F 0 "K_RCTL2" H 7900 4570 60  0000 C CNN
 F 1 "MX-1U" H 7900 4495 20  0000 C CNN
-F 2 "MX_Alps_Hybrid:MX-1U" H 7875 4420 60  0001 C CNN
+F 2 "MX_Alps_Hybrid:MX-1U-FLIPPED" H 7875 4420 60  0001 C CNN
 F 3 "" H 7875 4420 60  0001 C CNN
 	1    7900 4445
@@
 F 0 "K_SPACE1_3" H 3400 5095 60  0000 C CNN
 F 1 "MX-2.75U" H 3400 5020 20  0000 C CNN
-F 2 "MX_Alps_Hybrid:MX-2.75U" H 3375 4945 60  0001 C CNN
+F 2 "MX_Alps_Hybrid:MX-2.75U-ReversedStabilizers" H 3375 4945 60  0001 C CNN
 F 3 "" H 3375 4945 60  0001 C CNN
 	1    3400 4970
@@
 F 0 "K_SPACE3_3" H 5200 5095 60  0000 C CNN
 F 1 "MX-2.75U" H 5200 5020 20  0000 C CNN
-F 2 "MX_Alps_Hybrid:MX-2.75U" H 5175 4945 60  0001 C CNN
+F 2 "MX_Alps_Hybrid:MX-2.75U-ReversedStabilizers" H 5175 4945 60  0001 C CNN
 F 3 "" H 5175 4945 60  0001 C CNN
 	1    5200 4970
@@
 F 0 "K_RMOD2" H 6550 4570 60  0000 C CNN
 F 1 "MX-1U" H 6550 4495 20  0000 C CNN
-F 2 "MX_Alps_Hybrid:MX-1U" H 6525 4420 60  0001 C CNN
+F 2 "MX_Alps_Hybrid:MX-1U-FLIPPED" H 6525 4420 60  0001 C CNN
 F 3 "" H 6525 4420 60  0001 C CNN
 	1    6550 4445
@@
 F 0 "K_LALT2" H 2500 4580 60  0000 C CNN
 F 1 "MX-1.5U" H 2500 4505 20  0000 C CNN
-F 2 "MX_Alps_Hybrid:MX-1.5U" H 2475 4430 60  0001 C CNN
+F 2 "MX_Alps_Hybrid:MX-1.5U-FLIPPED" H 2475 4430 60  0001 C CNN
 F 3 "" H 2475 4430 60  0001 C CNN
 	1    2500 4455
@@
 F 0 "K_SPACE2_5" H 4300 6195 60  0000 C CNN
 F 1 "MX-1.25U" H 4300 6120 20  0000 C CNN
-F 2 "MX_Alps_Hybrid:MX-1.25U" H 4275 6045 60  0001 C CNN
+F 2 "MX_Alps_Hybrid:MX-1.25U-FLIPPED" H 4275 6045 60  0001 C CNN
 F 3 "" H 4275 6045 60  0001 C CNN
 	1    4300 6070

Commit message: Update: Bottom row to MX-Only footprints
Parts:
- K_LALT1, K_LGUI1, K_RALT1, K_RCTL1, K_RFN1: footprint MX_Alps_Hybrid:MX-1.25U -> MX_Alps_Hybrid:MXOnly-1.25U-FLIPPED
- K_LALT2: footprint MX_Alps_Hybrid:MX-1.5U-FLIPPED -> MX_Alps_Hybrid:MXOnly-1.5U
- K_LCTL1, K_RMOD1: footprint MX_Alps_Hybrid:MX-1.25U -> MX_Alps_Hybrid:MXOnly-1.25U
- K_LCTL2: footprint MX_Alps_Hybrid:MX-1.5U-FLIPPED -> MX_Alps_Hybrid:MXOnly-1.5U-FLIPPED
- K_LGUI2, K_RALT3, K_RCTL2, K_RMOD2: footprint MX_Alps_Hybrid:MX-1U-FLIPPED -> MX_Alps_Hybrid:MXOnly-1U
- K_RCTL3, K_SPACE2_4: footprint MX_Alps_Hybrid:MX-1.5U -> MX_Alps_Hybrid:MXOnly-1.5U
- K_RFN2, K_RFN3, K_RGUI1: footprint MX_Alps_Hybrid:MX-1U -> MX_Alps_Hybrid:MXOnly-1U
- K_RMOD3: footprint MX_Alps_Hybrid:MX-1.5U -> MX_Alps_Hybrid:MXOnly-1.5U-FLIPPED
- K_SPACE1_1: footprint MX_Alps_Hybrid:MX-2.25U-ReversedStabilizers -> MX_Alps_Hybrid:MXOnly-2.25U-ReversedStabilizers
- K_SPACE1_2: footprint MX_Alps_Hybrid:MX-2.75U-FLIPPED-ReversedStabilizers -> MX_Alps_Hybrid:MXOnly-2.75U-FLIPPED-ReversedStabilizers
- K_SPACE1_3, K_SPACE3_3: footprint MX_Alps_Hybrid:MX-2.75U-ReversedStabilizers -> MX_Alps_Hybrid:MXOnly-2.75U-ReversedStabilizers
- K_SPACE2_1, K_SPACE2_5: footprint MX_Alps_Hybrid:MX-1.25U-FLIPPED -> MX_Alps_Hybrid:MXOnly-1.25U-FLIPPED
- K_SPACE2_2: footprint MX_Alps_Hybrid:MX-6.25U-ReversedStabilizers -> MX_Alps_Hybrid:MXOnly-6.25U-ReversedStabilizers
- K_SPACE2_3: footprint MX_Alps_Hybrid:MX-7U-ReversedStabilizers -> MX_Alps_Hybrid:MXOnly-7U-ReversedStabilizers
- K_SPACE3_1: footprint MX_Alps_Hybrid:MX-2.75U-ReversedStabilizers -> MX_Alps_Hybrid:MXOnly-2.75U-FLIPPED-ReversedStabilizers
- K_SPACE3_2: footprint MX_Alps_Hybrid:MX-2.25U-FLIPPED-ReversedStabilizers -> MX_Alps_Hybrid:MXOnly-2.25U-ReversedStabilizers
Changed lines of the file:
@@
 F 0 "K_LCTL1" H 1550 3925 60  0000 C CNN
 F 1 "MX-1.25U" H 1550 3850 20  0000 C CNN
-F 2 "MX_Alps_Hybrid:MX-1.25U" H 1525 3775 60  0001 C CNN
+F 2 "MX_Alps_Hybrid:MXOnly-1.25U" H 1525 3775 60  0001 C CNN
 F 3 "" H 1525 3775 60  0001 C CNN
 	1    1550 3800
@@
 F 0 "K_LGUI1" H 2050 3925 60  0000 C CNN
 F 1 "MX-1.25U" H 2050 3850 20  0000 C CNN
-F 2 "MX_Alps_Hybrid:MX-1.25U" H 2025 3775 60  0001 C CNN
+F 2 "MX_Alps_Hybrid:MXOnly-1.25U-FLIPPED" H 2025 3775 60  0001 C CNN
 F 3 "" H 2025 3775 60  0001 C CNN
 	1    2050 3800
@@
 F 0 "K_LALT1" H 2500 3925 60  0000 C CNN
 F 1 "MX-1.25U" H 2500 3850 20  0000 C CNN
-F 2 "MX_Alps_Hybrid:MX-1.25U" H 2475 3775 60  0001 C CNN
+F 2 "MX_Alps_Hybrid:MXOnly-1.25U-FLIPPED" H 2475 3775 60  0001 C CNN
 F 3 "" H 2475 3775 60  0001 C CNN
 	1    2500 3800
@@
 F 0 "K_LCTL2" H 1550 4580 60  0000 C CNN
 F 1 "MX-1.5U" H 1550 4505 20  0000 C CNN
-F 2 "MX_Alps_Hybrid:MX-1.5U-FLIPPED" H 1525 4430 60  0001 C CNN
+F 2 "MX_Alps_Hybrid:MXOnly-1.5U-FLIPPED" H 1525 4430 60  0001 C CNN
 F 3 "" H 1525 4430 60  0001 C CNN
 	1    1550 4455
@@
 F 0 "K_LGUI2" H 2050 4580 60  0000 C CNN
 F 1 "MX-1U" H 2050 4505 20  0000 C CNN
-F 2 "MX_Alps_Hybrid:MX-1U-FLIPPED" H 2025 4430 60  0001 C CNN
+F 2 "MX_Alps_Hybrid:MXOnly-1U" H 2025 4430 60  0001 C CNN
 F 3 "" H 2025 4430 60  0001 C CNN
 	1    2050 4455
@@
 F 0 "K_SPACE1_1" H 3400 3925 60  0000 C CNN
 F 1 "MX-2.25U" H 3400 3850 20  0000 C CNN
-F 2 "MX_Alps_Hybrid:MX-2.25U-ReversedStabilizers" H 3375 3775 60  0001 C CNN
+F 2 "MX_Alps_Hybrid:MXOnly-2.25U-ReversedStabilizers" H 3375 3775 60  0001 C CNN
 F 3 "" H 3375 3775 60  0001 C CNN
 	1    3400 3800
@@
 F 0 "K_SPACE2_1" H 4300 3925 60  0000 C CNN
 F 1 "MX-1.25U" H 4300 3850 20  0000 C CNN
-F 2 "MX_Alps_Hybrid:MX-1.25U-FLIPPED" H 4275 3775 60  0001 C CNN
+F 2 "MX_Alps_Hybrid:MXOnly-1.25U-FLIPPED" H 4275 3775 60  0001 C CNN
 F 3 "" H 4275 3775 60  0001 C CNN
 	1    4300 3800
@@
 F 0 "K_SPACE3_1" H 5200 3925 60  0000 C CNN
 F 1 "MX-2.75U" H 5200 3850 20  0000 C CNN
-F 2 "MX_Alps_Hybrid:MX-2.75U-ReversedStabilizers" H 5175 3775 60  0001 C CNN
+F 2 "MX_Alps_Hybrid:MXOnly-2.75U-FLIPPED-ReversedStabilizers" H 5175 3775 60  0001 C CNN
 F 3 "" H 5175 3775 60  0001 C CNN
 	1    5200 3800
@@
 F 0 "K_SPACE1_2" H 3400 4575 60  0000 C CNN
 F 1 "MX-2.75U" H 3400 4500 20  0000 C CNN
-F 2 "MX_Alps_Hybrid:MX-2.75U-FLIPPED-ReversedStabilizers" H 3375 4425 60  0001 C CNN
+F 2 "MX_Alps_Hybrid:MXOnly-2.75U-FLIPPED-ReversedStabilizers" H 3375 4425 60  0001 C CNN
 F 3 "" H 3375 4425 60  0001 C CNN
 	1    3400 4450
@@
 F 0 "K_SPACE3_2" H 5200 4575 60  0000 C CNN
 F 1 "MX-2.25U" H 5200 4500 20  0000 C CNN
-F 2 "MX_Alps_Hybrid:MX-2.25U-FLIPPED-ReversedStabilizers" H 5175 4425 60  0001 C CNN
+F 2 "MX_Alps_Hybrid:MXOnly-2.25U-ReversedStabilizers" H 5175 4425 60  0001 C CNN
 F 3 "" H 5175 4425 60  0001 C CNN
 	1    5200 4450
@@
 F 0 "K_SPACE2_2" H 4300 4575 60  0000 C CNN
 F 1 "MX-6.25U" H 4300 4500 20  0000 C CNN
-F 2 "MX_Alps_Hybrid:MX-6.25U-ReversedStabilizers" H 4275 4425 60  0001 C CNN
+F 2 "MX_Alps_Hybrid:MXOnly-6.25U-ReversedStabilizers" H 4275 4425 60  0001 C CNN
 F 3 "" H 4275 4425 60  0001 C CNN
 	1    4300 4450
@@
 F 0 "K_RALT1" H 6100 3925 60  0000 C CNN
 F 1 "MX-1.25U" H 6100 3850 20  0000 C CNN
-F 2 "MX_Alps_Hybrid:MX-1.25U" H 6075 3775 60  0001 C CNN
+F 2 "MX_Alps_Hybrid:MXOnly-1.25U-FLIPPED" H 6075 3775 60  0001 C CNN
 F 3 "" H 6075 3775 60  0001 C CNN
 	1    6100 3800
@@
 F 0 "K_RALT3" H 6100 5075 60  0000 C CNN
 F 1 "MX-1U" H 6100 5000 20  0000 C CNN
-F 2 "MX_Alps_Hybrid:MX-1U-FLIPPED" H 6075 4925 60  0001 C CNN
+F 2 "MX_Alps_Hybrid:MXOnly-1U" H 6075 4925 60  0001 C CNN
 F 3 "" H 6075 4925 60  0001 C CNN
 	1    6100 4950
@@
 F 0 "K_RMOD1" H 6550 3925 60  0000 C CNN
 F 1 "MX-1.25U" H 6550 3850 20  0000 C CNN
-F 2 "MX_Alps_Hybrid:MX-1.25U" H 6525 3775 60  0001 C CNN
+F 2 "MX_Alps_Hybrid:MXOnly-1.25U" H 6525 3775 60  0001 C CNN
 F 3 "" H 6525 3775 60  0001 C CNN
 	1    6550 3800
@@
 F 0 "K_RGUI1" H 7000 3925 60  0000 C CNN
 F 1 "MX-1U" H 7000 3850 20  0000 C CNN
-F 2 "MX_Alps_Hybrid:MX-1U" H 6975 3775 60  0001 C CNN
+F 2 "MX_Alps_Hybrid:MXOnly-1U" H 6975 3775 60  0001 C CNN
 F 3 "" H 6975 3775 60  0001 C CNN
 	1    7000 3800
@@
 F 0 "K_RFN1" H 7450 3925 60  0000 C CNN
 F 1 "MX-1.25U" H 7450 3850 20  0000 C CNN
-F 2 "MX_Alps_Hybrid:MX-1.25U" H 7425 3775 60  0001 C CNN
+F 2 "MX_Alps_Hybrid:MXOnly-1.25U-FLIPPED" H 7425 3775 60  0001 C CNN
 F 3 "" H 7425 3775 60  0001 C CNN
 	1    7450 3800
@@
 F 0 "K_RCTL1" H 7900 3925 60  0000 C CNN
 F 1 "MX-1.25U" H 7900 3850 20  0000 C CNN
-F 2 "MX_Alps_Hybrid:MX-1.25U" H 7875 3775 60  0001 C CNN
+F 2 "MX_Alps_Hybrid:MXOnly-1.25U-FLIPPED" H 7875 3775 60  0001 C CNN
 F 3 "" H 7875 3775 60  0001 C CNN
 	1    7900 3800
@@
 F 0 "K_SPACE2_3" H 4300 5095 60  0000 C CNN
 F 1 "MX-7U" H 4300 5020 20  0000 C CNN
-F 2 "MX_Alps_Hybrid:MX-7U-ReversedStabilizers" H 4275 4945 60  0001 C CNN
+F 2 "MX_Alps_Hybrid:MXOnly-7U-ReversedStabilizers" H 4275 4945 60  0001 C CNN
 F 3 "" H 4275 4945 60  0001 C CNN
 	1    4300 4970
@@
 F 0 "K_RFN2" H 7450 4570 60  0000 C CNN
 F 1 "MX-1U" H 7450 4495 20  0000 C CNN
-F 2 "MX_Alps_Hybrid:MX-1U" H 7425 4420 60  0001 C CNN
+F 2 "MX_Alps_Hybrid:MXOnly-1U" H 7425 4420 60  0001 C CNN
 F 3 "" H 7425 4420 60  0001 C CNN
 	1    7450 4445
@@
 F 0 "K_RCTL2" H 7900 4570 60  0000 C CNN
 F 1 "MX-1U" H 7900 4495 20  0000 C CNN
-F 2 "MX_Alps_Hybrid:MX-1U-FLIPPED" H 7875 4420 60  0001 C CNN
+F 2 "MX_Alps_Hybrid:MXOnly-1U" H 7875 4420 60  0001 C CNN
 F 3 "" H 7875 4420 60  0001 C CNN
 	1    7900 4445
@@
 F 0 "K_SPACE2_4" H 4300 5615 60  0000 C CNN
 F 1 "MX-1.5U" H 4300 5540 20  0000 C CNN
-F 2 "MX_Alps_Hybrid:MX-1.5U" H 4275 5465 60  0001 C CNN
+F 2 "MX_Alps_Hybrid:MXOnly-1.5U" H 4275 5465 60  0001 C CNN
 F 3 "" H 4275 5465 60  0001 C CNN
 	1    4300 5490
@@
 F 0 "K_SPACE1_3" H 3400 5095 60  0000 C CNN
 F 1 "MX-2.75U" H 3400 5020 20  0000 C CNN
-F 2 "MX_Alps_Hybrid:MX-2.75U-ReversedStabilizers" H 3375 4945 60  0001 C CNN
+F 2 "MX_Alps_Hybrid:MXOnly-2.75U-ReversedStabilizers" H 3375 4945 60  0001 C CNN
 F 3 "" H 3375 4945 60  0001 C CNN
 	1    3400 4970
@@
 F 0 "K_SPACE3_3" H 5200 5095 60  0000 C CNN
 F 1 "MX-2.75U" H 5200 5020 20  0000 C CNN
-F 2 "MX_Alps_Hybrid:MX-2.75U-ReversedStabilizers" H 5175 4945 60  0001 C CNN
+F 2 "MX_Alps_Hybrid:MXOnly-2.75U-ReversedStabilizers" H 5175 4945 60  0001 C CNN
 F 3 "" H 5175 4945 60  0001 C CNN
 	1    5200 4970
@@
 F 0 "K_RMOD2" H 6550 4570 60  0000 C CNN
 F 1 "MX-1U" H 6550 4495 20  0000 C CNN
-F 2 "MX_Alps_Hybrid:MX-1U-FLIPPED" H 6525 4420 60  0001 C CNN
+F 2 "MX_Alps_Hybrid:MXOnly-1U" H 6525 4420 60  0001 C CNN
 F 3 "" H 6525 4420 60  0001 C CNN
 	1    6550 4445
@@
 F 0 "K_RMOD3" H 6550 5075 60  0000 C CNN
 F 1 "MX-1.5U" H 6550 5000 20  0000 C CNN
-F 2 "MX_Alps_Hybrid:MX-1.5U" H 6525 4925 60  0001 C CNN
+F 2 "MX_Alps_Hybrid:MXOnly-1.5U-FLIPPED" H 6525 4925 60  0001 C CNN
 F 3 "" H 6525 4925 60  0001 C CNN
 	1    6550 4950
@@
 F 0 "K_RFN3" H 7450 5075 60  0000 C CNN
 F 1 "MX-1U" H 7450 5000 20  0000 C CNN
-F 2 "MX_Alps_Hybrid:MX-1U" H 7425 4925 60  0001 C CNN
+F 2 "MX_Alps_Hybrid:MXOnly-1U" H 7425 4925 60  0001 C CNN
 F 3 "" H 7425 4925 60  0001 C CNN
 	1    7450 4950
@@
 F 0 "K_RCTL3" H 7895 5075 60  0000 C CNN
 F 1 "MX-1.5U" H 7895 5000 20  0000 C CNN
-F 2 "MX_Alps_Hybrid:MX-1.5U" H 7870 4925 60  0001 C CNN
+F 2 "MX_Alps_Hybrid:MXOnly-1.5U" H 7870 4925 60  0001 C CNN
 F 3 "" H 7870 4925 60  0001 C CNN
 	1    7895 4950
@@
 F 0 "K_LALT2" H 2500 4580 60  0000 C CNN
 F 1 "MX-1.5U" H 2500 4505 20  0000 C CNN
-F 2 "MX_Alps_Hybrid:MX-1.5U-FLIPPED" H 2475 4430 60  0001 C CNN
+F 2 "MX_Alps_Hybrid:MXOnly-1.5U" H 2475 4430 60  0001 C CNN
 F 3 "" H 2475 4430 60  0001 C CNN
 	1    2500 4455
@@
 F 0 "K_SPACE2_5" H 4300 6195 60  0000 C CNN
 F 1 "MX-1.25U" H 4300 6120 20  0000 C CNN
-F 2 "MX_Alps_Hybrid:MX-1.25U-FLIPPED" H 4275 6045 60  0001 C CNN
+F 2 "MX_Alps_Hybrid:MXOnly-1.25U-FLIPPED" H 4275 6045 60  0001 C CNN
 F 3 "" H 4275 6045 60  0001 C CNN
 	1    4300 6070

Commit message: Update: Switch most of remaining switches to MX-only
There isn't an MX-only footprint for ISO enter, so that one
is still MX and Alps. When I have a chance, I'll make an MX-only
version of it.
Parts:
- K_#0_1, K_#1, K_#2, K_#3, K_#4, K_#5, K_#6, K_#7, K_#8, K_#9, K_'1, K_,1, K_-1, K_.1, K_;1, K_=1, K_A1, K_B1, K_BACK1, K_BACK2, K_C1, K_D1, K_DEL1, K_E1, K_ESC1, K_F1, K_FN1, K_G1, K_H1, K_I1, K_ISO#1, K_ISO\1, K_J1, K_K1, K_L1, K_M1, K_N1, K_O1, K_P1, K_Q1, K_R1, K_RSHIFT2, K_S1, K_T1, K_U1, K_V1, K_W1, K_X1, K_Y1, K_Z1, K_[1, K_\1, K_]1: footprint MX_Alps_Hybrid:MX-1U -> MX_Alps_Hybrid:MXOnly-1U
- K_CAPS1, K_FN2, K_RSHIFT3: footprint MX_Alps_Hybrid:MX-1.75U -> MX_Alps_Hybrid:MXOnly-1.75U
- K_CAPS2: footprint MX_Alps_Hybrid:MX-1.25U-FLIPPED -> MX_Alps_Hybrid:MXOnly-1.25U-FLIPPED
- K_ENTER1, K_LSHIFT1: footprint MX_Alps_Hybrid:MX-2.25U -> MX_Alps_Hybrid:MXOnly-2.25U
- K_LSHIFT2: footprint MX_Alps_Hybrid:MX-1.25U -> MX_Alps_Hybrid:MXOnly-1.25U
- K_RSHIFT1: footprint MX_Alps_Hybrid:MX-2.75U-FLIPPED -> MX_Alps_Hybrid:MXOnly-2.75U
- K_TAB1: footprint MX_Alps_Hybrid:MX-1.5U -> MX_Alps_Hybrid:MXOnly-1.5U

Commit message: Update: Simplify right shift, fix footprint errors, layout switches
Parts:
- removed K_FN2: MX-1.75U, MX_Alps_Hybrid:MXOnly-1.75U, symbol MX-1.75U
- added D57: D_Small, Diodes_SMD:D_SOD-123, symbol D_Small
- added R57: 820, Resistors_SMD:R_0603, symbol R_Small
- K_BACK1: footprint MX_Alps_Hybrid:MXOnly-1U -> MX_Alps_Hybrid:MXOnly-2U
- K_ISOENTER1: footprint MX_Alps_Hybrid:MX-ISO -> MX_Alps_Hybrid:MXOnly-ISO-ReversedStabilizers
- K_\1: value MX-1U -> MX-1.5U; footprint MX_Alps_Hybrid:MXOnly-1U -> MX_Alps_Hybrid:MXOnly-1.5U; symbol MX-1U -> MX-1.5U
- renumbered D57 to D58, D58 to D59, D59 to D60, D60 to D61, D61 to D62, D62 to D63, D63 to D64, D64 to D65, D65 to D66, D66 to D67, D67 to D68, K_FN1 to K_/1, K_RSHIFT2 to K_FN1, K_RSHIFT3 to K_RSHIFT2, R57 to R58, R58 to R59, R59 to R60, R60 to R61, R61 to R62, R62 to R63, R63 to R64, R64 to R65, R65 to R66, R66 to R67, R67 to R68
Connections:
- net COL11: no longer K_'1.1 (COL), K_=1.1 (COL), K_RGUI1.1 (COL), K_[1.1 (COL)
- net COL13: no longer K_FN1.1 (COL)
- net COL14: now also K_FN1.1 (COL)
- net ROW3: now also D57.1 (K)
- net VCC: now also R57.2
- net at D56.2 (A), K_RSHIFT1.2 (ROW), K_RSHIFT2.2 (ROW): no longer K_FN1.2 (ROW)
- net at K_RSHIFT1.3 (LED), K_RSHIFT2.3 (LED), R56.1: no longer K_FN1.3 (LED)
- new net: D57.2 (A), K_FN1.2 (ROW)
- new net: K_FN1.3 (LED), R57.1
- new net COL12: K_'1.1 (COL), K_=1.1 (COL), K_RGUI1.1 (COL), K_[1.1 (COL)
Other:
- moved on the sheet: K_RSHIFT2
