File: co60.sch (KiCad schematic (older format))
At the start: 23 parts, among them J1 Conn_01x06, Q1 FMMT493TA, SW1 SW_Push, U1 ATMEGA32U4, Y1 16MHz

Commit message: Update: Add more info to BOM, and reformat it
Parts:
- C1: Digi-Key_PN (none) -> 478-1167-1-ND
- C3: Digi-Key_PN (none) -> 445-13234-1-ND
- C4: Digi-Key_PN (none) -> 445-2500-1-ND
- C8: Digi-Key_PN (none) -> 1276-1900-1-ND
- DP1: Digi-Key_PN (none) -> 1727-3884-1-ND
- F1: Digi-Key_PN (none) -> F2772CT-ND
- RC1: Digi-Key_PN (none) -> 311-1.5KGRCT-ND
- RC2: Digi-Key_PN (none) -> P10KGCT-ND
- RC4: Digi-Key_PN (none) -> 311-22GRCT-ND
- RC6: Digi-Key_PN (none) -> RMCF0603JT5K10CT-ND
- SW1: Digi-Key_PN (none) -> EG2531CT-ND
- U1: Digi-Key_PN (none) -> ATMEGA32U4-AURCT-ND
- USB1: Digi-Key_PN (none) -> 12401598E4#2ACT-ND
- Y1: Digi-Key_PN (none) -> 644-1168-1-ND
Changed lines of the file:
@@
 F 3 "http://datasheets.avx.com/C0GNP0-Dielectric.pdf" H 6470 2980 50  0001 C CNN
 F 4 "06035A220JAT2A" H 6470 2980 60  0001 C CNN "Product"
+F 5 "478-1167-1-ND" H 6470 2980 60  0001 C CNN "Digi-Key_PN"
 	1    6470 2980
 	1    0    0    -1
@@
 F 3 "https://product.tdk.com/info/en/catalog/datasheets/mlcc_commercial_lowprofile_en.pdf" H 6675 5705 50  0001 C CNN
 F 4 "CGB3B3JB1C105K055AB" H 6675 5705 60  0001 C CNN "Product"
+F 5 "445-13234-1-ND" H 6675 5705 60  0001 C CNN "Digi-Key_PN"
 	1    6675 5705
 	1    0    0    -1
@@
 F 3 "https://product.tdk.com/info/en/catalog/datasheets/mlcc_commercial_hightemp_en.pdf" H 1150 1050 50  0001 C CNN
 F 4 "C1608X8R1E104K080AA" H 1150 1050 60  0001 C CNN "Product"
+F 5 "445-2500-1-ND" H 1150 1050 60  0001 C CNN "Digi-Key_PN"
 	1    1150 1050
 	1    0    0    -1
@@
 F 3 "http://www.samsungsem.com/kr/support/product-search/mlcc/__icsFiles/afieldfile/2016/12/21/CL10A475KA8NQNC_161221.pdf" H 900 1050 50  0001 C CNN
 F 4 "CL10A475KA8NQNC" H 900 1050 60  0001 C CNN "Product"
+F 5 "1276-1900-1-ND" H 900 1050 60  0001 C CNN "Digi-Key_PN"
 	1    900  1050
 	1    0    0    -1
@@
 F 1 "10k" V 9765 4905 50  0000 C CNN
 F 2 "Resistors_SMD:R_0603" V 9695 4905 50  0001 C CNN
-F 3 "" H 9765 4905 50  0001 C CNN
+F 3 "https://industrial.panasonic.com/ww/products/resistors/chip-resistors/general-purpose-chip-resistors/thick-film-chip-resistors/ERJ3GEYJ103V" H 9765 4905 50  0001 C CNN
 F 4 "ERJ-3GEYJ103V" V 9765 4905 60  0001 C CNN "Product"
+F 5 "P10KGCT-ND" V 9765 4905 60  0001 C CNN "Digi-Key_PN"
 	1    9765 4905
 	1    0    0    -1
@@
 F 1 "22" V 4510 3605 50  0000 C CNN
 F 2 "Resistors_SMD:R_0603" V 4440 3605 50  0001 C CNN
-F 3 "" H 4510 3605 50  0001 C CNN
+F 3 "http://www.yageo.com/documents/recent/PYu-RC_Group_51_RoHS_L_9.pdf" H 4510 3605 50  0001 C CNN
 F 4 "RC0603JR-0722RL" V 4510 3605 60  0001 C CNN "Product"
+F 5 "311-22GRCT-ND" V 4510 3605 60  0001 C CNN "Digi-Key_PN"
 	1    4510 3605
 	0    1    1    0
@@
 F 1 "5.1k" V 3335 3245 50  0000 C CNN
 F 2 "Resistors_SMD:R_0603" V 3265 3245 50  0001 C CNN
-F 3 "" H 3335 3245 50  0001 C CNN
+F 3 "https://www.seielect.com/Catalog/SEI-RMCF_RMCP.pdf" H 3335 3245 50  0001 C CNN
 F 4 "RMCF0603JT5K10" V 3335 3245 60  0001 C CNN "Product"
+F 5 "RMCF0603JT5K10CT-ND" V 3335 3245 60  0001 C CNN "Digi-Key_PN"
 	1    3335 3245
 	0    1    1    0
@@
 F 4 "TL3342F160QG/TR" H 6685 2230 60  0001 C CNN "Product"
 F 5 "https://www.digikey.ca/product-detail/en/e-switch/TL3342F160QG-TR/EG2531CT-ND/379004" H 6685 2230 60  0001 C CNN "DigiKey Page"
+F 6 "EG2531CT-ND" H 6685 2230 60  0001 C CNN "Digi-Key_PN"
 	1    6685 2230
 	1    0    0    -1
@@
 F 1 "1.5k" H 4395 1040 50  0000 L CNN
 F 2 "Resistors_SMD:R_0603" H 4365 1080 50  0001 C CNN
-F 3 "" H 4365 1080 50  0001 C CNN
+F 3 "http://www.yageo.com/documents/recent/PYu-RC_Group_51_RoHS_L_9.pdf" H 4365 1080 50  0001 C CNN
 F 4 "RC0603JR-071K5L" H 4365 1080 60  0001 C CNN "Product"
+F 5 "311-1.5KGRCT-ND" H 4365 1080 60  0001 C CNN "Digi-Key_PN"
 	1    4365 1080
 	0    1    1    0
@@
 F 3 "http://ww1.microchip.com/downloads/en/DeviceDoc/Atmel-7766-8-bit-AVR-ATmega16U4-32U4_Summary.pdf" H 8140 3930 60  0001 C CNN
 F 4 "Microcontroller" H 8140 3930 60  0001 C CNN "Description"
+F 5 "ATMEGA32U4-AURCT-ND" H 8140 3930 60  0001 C CNN "Digi-Key_PN"
 	1    8140 3930
 	1    0    0    -1
@@
 F 3 "https://www.digikey.com/product-detail/en/ndk-america-inc/NX2520SA-16MHZ-STD-CSW-4/644-1168-1-ND/3125557" H 6770 2630 50  0001 C CNN
 F 4 "NX2520SA-16MHZ-STD-CSW-4" H 6770 2630 60  0001 C CNN "Product"
+F 5 "644-1168-1-ND" H 6770 2630 60  0001 C CNN "Digi-Key_PN"
 	1    6770 2630
 	-1   0    0    1
@@
 F 3 "https://assets.nexperia.com/documents/data-sheet/PRTR5V0U2X.pdf" H 4335 4270 50  0001 C CNN
 F 4 "Rail-to-rail ESD protection circuitry" H 4285 4320 60  0001 C CNN "Description"
+F 5 "1727-3884-1-ND" H 4285 4320 60  0001 C CNN "Digi-Key_PN"
 	1    4285 4320
 	1    0    0    -1
@@
 F 3 "http://www.littelfuse.com/~/media/electronics/datasheets/resettable_ptcs/littelfuse_ptc_0805l_datasheet.pdf.pdf" H 3410 2850 50  0001 C CNN
 F 4 "0805L050WR" V 3410 2850 60  0001 C CNN "Product"
+F 5 "F2772CT-ND" V 3410 2850 60  0001 C CNN "Digi-Key_PN"
 	1    3410 2850
 	0    1    1    0
@@
 F 3 "https://media.digikey.com/pdf/Data%20Sheets/Amphenol%20PDFs/12401598E4%232A_Dwg.pdf" H 1700 3450 60  0001 C CNN
 F 4 "USB Type-C connector" H 2400 3400 60  0001 C CNN "Description"
+F 5 "12401598E4#2ACT-ND" H 2400 3400 60  0001 C CNN "Digi-Key_PN"
 	1    2400 3400
 	1    0    0    -1

Commit message: Update: More BOM work
Parts:
- DP1: Product (none) -> PRTR5V0U2X
- Q1: Product (none) -> FMMT493TA
- U1: Product (none) -> ATMEGA32U4-AU
- USB1: Product (none) -> 12401598E4#2A
Changed lines of the file:
@@
 F 4 "Microcontroller" H 8140 3930 60  0001 C CNN "Description"
 F 5 "ATMEGA32U4-AURCT-ND" H 8140 3930 60  0001 C CNN "Digi-Key_PN"
+F 6 "ATMEGA32U4-AU" H 8140 3930 60  0001 C CNN "Product"
 	1    8140 3930
 	1    0    0    -1
@@
 F 4 "Rail-to-rail ESD protection circuitry" H 4285 4320 60  0001 C CNN "Description"
 F 5 "1727-3884-1-ND" H 4285 4320 60  0001 C CNN "Digi-Key_PN"
+F 6 "PRTR5V0U2X" H 4285 4320 60  0001 C CNN "Product"
 	1    4285 4320
 	1    0    0    -1
@@
 F 4 "USB Type-C connector" H 2400 3400 60  0001 C CNN "Description"
 F 5 "12401598E4#2ACT-ND" H 2400 3400 60  0001 C CNN "Digi-Key_PN"
+F 6 "12401598E4#2A" H 2400 3400 60  0001 C CNN "Product"
 	1    2400 3400
 	1    0    0    -1
@@
 F 11 "Diodes Incorporated" H 5115 2180 60  0001 L CNN "Manufacturer"
 F 12 "Active" H 5115 2280 60  0001 L CNN "Status"
+F 13 "FMMT493TA" H 4915 1080 60  0001 C CNN "Product"
 	1    4915 1080
 	1    0    0    -1

Commit message: Update: More work on BOM
Parts:
- DP1: Product PRTR5V0U2X -> PRTR5V0U2X,215
Changed lines of the file:
@@
 F 4 "Rail-to-rail ESD protection circuitry" H 4285 4320 60  0001 C CNN "Description"
 F 5 "1727-3884-1-ND" H 4285 4320 60  0001 C CNN "Digi-Key_PN"
-F 6 "PRTR5V0U2X" H 4285 4320 60  0001 C CNN "Product"
+F 6 "PRTR5V0U2X,215" H 4285 4320 60  0001 C CNN "Product"
 	1    4285 4320
 	1    0    0    -1

Commit message: Fix: Transistor base and emitter pin assignments were flipped
In the inital version of the digikey footprint library that I
was using, the pin assignments were wrong on the transistor
schematic. This lead me to wiring up the emitter to where the
base was supposed to go and vice versa. As a result, backlighting
will not work on any revision of the board prior to this commit.
This commit updates the digikey library, which has the fixed
pin assignments, and re-routes the transistor pads correctly.
Changed lines of the file:
@@
 Connection ~ 1570 3950
-Wire Wire Line
-	4465 1080 4565 1080
-Wire Wire Line
-	4915 685  5015 685
-Wire Wire Line
-	5015 685  5015 780
-Wire Wire Line
-	5015 1380 5015 1485
 Wire Wire Line
 	6920 2630 7140 2630
@@
 Wire Wire Line
 	7140 3575 7140 3030
+Wire Wire Line
+	4465 1080 4715 1080
+Wire Wire Line
+	4915 685  5015 685
+Wire Wire Line
+	5015 685  5015 880
+Wire Wire Line
+	5015 1280 5015 1485
 $EndSCHEMATC

Commit message: Update: Migrate project to Kicad 5
Parts:
- C1, C2, C3, C4, C5, C6, C7, C8: symbol C -> co60-rescue:C
- DP1: symbol PRTR5V0U2X -> co60-rescue:PRTR5V0U2X
- F1: symbol Polyfuse_Small -> co60-rescue:Polyfuse_Small
- J1: symbol Conn_01x06 -> co60-rescue:Conn_01x06
- Q1: symbol FMMT493TA -> dk_Transistors-Bipolar-BJT-Single:FMMT493TA
- RC1: symbol R_Small -> co60-rescue:R_Small
- RC2, RC3, RC4, RC5, RC6, RC7: symbol R -> co60-rescue:R
- SW1: symbol SW_Push -> co60-rescue:SW_Push
- U1: symbol ATMEGA32U4 -> atmega32u4:ATMEGA32U4
- USB1: symbol 12401598E4#2A -> Type-C:12401598E4#2A
- Y1: symbol Crystal_GND24 -> co60-rescue:Crystal_GND24
Connections:
- wire segments 143 -> 179

Commit message: Update: Switch USB connector from Amphenol to Korean HRO
This connector is smaller, and I believe it will interfere less with the
switches when they are installed.
Parts:
- removed DP1: PRTR5V0U2X, locallib:SOT143B, symbol co60-rescue:PRTR5V0U2X
- removed USB1: 12401598E4#2A, Type-C:12401598E4#2A, symbol Type-C:12401598E4#2A
- added ESD1: PRTR5V0U2X, locallib:SOT143B, symbol co60-rescue:PRTR5V0U2X
- added USB1: HRO-TYPE-C-31-M-12, Type-C:HRO-TYPE-C-31-M-12, symbol Type-C:HRO-TYPE-C-31-M-12
Connections:
- wire segments 179 -> 157
- no-connect marks 15 -> 7

Commit message: Update: HRO connector to newest footprint version
This version has solder pads for the through hole legs,
which are necessary when doing PCB assembly.
Parts:
- USB1: footprint Type-C:HRO-TYPE-C-31-M-12 -> Type-C:HRO-TYPE-C-31-M-12-Assembly
Changed lines of the file:
@@
 F 0 "USB1" H 2321 4672 60  0000 C CNN
 F 1 "HRO-TYPE-C-31-M-12" H 2321 4566 60  0000 C CNN
-F 2 "Type-C:HRO-TYPE-C-31-M-12" H 2490 3875 60  0001 C CNN
+F 2 "Type-C:HRO-TYPE-C-31-M-12-Assembly" H 2490 3875 60  0001 C CNN
 F 3 "" H 2490 3875 60  0001 C CNN
 	1    2490 3875

Commit message: Update: Initial work on switching to STM32
The schematic is complete, though may need revising.
The PCB components need to be placed and routed.
Parts:
- removed J1: Conn_01x06, Socket_Strips:Socket_Strip_Straight_1x06_Pitch2.54mm, symbol co60-rescue:Conn_01x06
- removed RC2, RC3: 10k, Resistors_SMD:R_0603, symbol co60-rescue:R
- removed U1: ATMEGA32U4, tqfp:TQFP44, symbol atmega32u4:ATMEGA32U4
- added C10, C11: 1u, Capacitors_SMD:C_0603, symbol co60-rescue:C
- added C9: 100n, Capacitors_SMD:C_0603, symbol co60-rescue:C
- added RC8: 10k, Resistors_SMD:R_0603, symbol co60-rescue:R
- added RC9: 1.5k, Resistors_SMD:R_0603, symbol co60-rescue:R_Small
- added U1: STM32F303CBTx, Housings_QFP:LQFP-48_7x7mm_Pitch0.5mm, symbol MCU_ST_STM32F3:STM32F303CBTx
- added U2: TLV70233_SOT23-5, TO_SOT_Packages_SMD:SOT-23-5, symbol Regulator_Linear:TLV70233_SOT23-5
- C1: value 22p -> 30p; Digi-Key_PN 478-1167-1-ND -> (none); LCSC PN (none) -> C22397
- C2: value 22p -> 30p
- C3: value 1u -> 100n; Digi-Key_PN 445-13234-1-ND -> 445-2500-1-ND; Product CGB3B3JB1C105K055AB -> C1608X8R1E104K080AA
- C5: value 100n -> 4.7u; Digi-Key_PN (none) -> 1276-1900-1-ND; Product C1608X8R1E104K080AA -> CL10A475KA8NQNC
- C6: value 100n -> 1u; Digi-Key_PN (none) -> 445-13234-1-ND; Product C1608X8R1E104K080AA -> CGB3B3JB1C105K055AB
- C7: value 100n -> 10n; Product C1608X8R1E104K080AA -> (none)
- C8: value 4.7u -> 100n; Digi-Key_PN 1276-1900-1-ND -> 445-2500-1-ND; Product CL10A475KA8NQNC -> C1608X8R1E104K080AA
- Y1: value 16MHz -> 8MHz; footprint Crystals:Crystal_SMD_2520-4pin_2.5x2.0mm -> Crystals:Crystal_SMD_5032-4pin_5.0x3.2mm; Digi-Key_PN 644-1168-1-ND -> (none); LCSC PN (none) -> C133333; Product NX2520SA-16MHZ-STD-CSW-4 -> Zhejiang Abel Elec SMD-5032_4P8M20pf20ppm
Connections:
- net labels added: +3.3V, +5V, OSC_IN, OSC_OUT
- wire segments 157 -> 164
- no-connect marks 7 -> 14
Other:
- moved on the sheet: C1, C2, ESD1, F1, RC4, RC5, RC6, RC7, USB1, Y1
