File: rgb_underglow.sch (KiCad schematic (older format))
At the start: 33 parts, among them U4 SN74LV1T34DBVR

Commit message: Update: Work on routing RGB LEDs
Parts:
- added RC9: 500, Resistor_SMD:R_0603_1608Metric, symbol co60-rescue:R
Connections:
- net RGBLED: now also RC9.1; no longer U4.4 (Y)
- new net: RC9.2, U4.4 (Y)
Changed lines of the file:
@@
 Wire Wire Line
 	8720 3500 8720 3650
-Text GLabel 8935 3300 2    50   Input ~ 0
+Text GLabel 9235 3300 2    50   Input ~ 0
 RGBLED
-Wire Wire Line
-	8600 3300 8935 3300
 Text GLabel 7640 3300 0    50   Input ~ 0
 RGBLED_3V3
@@
 	7900 1150 8300 1150
 NoConn ~ 5400 4600
+$Comp
+L co60-rescue:R RC9
+U 1 1 5C33F401
+P 8915 3300
+F 0 "RC9" V 8708 3300 50  0000 C CNN
+F 1 "500" V 8799 3300 50  0000 C CNN
+F 2 "Resistor_SMD:R_0603_1608Metric" V 8845 3300 50  0001 C CNN
+F 3 "" H 8915 3300 50  0001 C CNN
+	1    8915 3300
+	0    1    1    0
+$EndComp
+Wire Wire Line
+	8600 3300 8765 3300
+Wire Wire Line
+	9065 3300 9235 3300
 $EndSCHEMATC

Commit message: Update: Improve crystal routing
Parts:
- RC9: value 500 -> 470; LCSC PN (none) -> C114433
Changed lines of the file:
@@
 P 8915 3300
 F 0 "RC9" V 8708 3300 50  0000 C CNN
-F 1 "500" V 8799 3300 50  0000 C CNN
+F 1 "470" V 8799 3300 50  0000 C CNN
 F 2 "Resistor_SMD:R_0603_1608Metric" V 8845 3300 50  0001 C CNN
 F 3 "" H 8915 3300 50  0001 C CNN
+F 4 "C114433" V 8915 3300 50  0001 C CNN "LCSC PN"
 	1    8915 3300
 	0    1    1    0

Commit message: Update: schematic cleanup
Parts:
- C12, C13, C14, C15, C16, C17, C18, C19, C20, C21, C22, C23, C24, C25, C26, C27: value 0.1uF -> 100n; LCSC PN (none) -> C1590
Changed lines of the file:
@@
 P 6700 1300
 F 0 "C12" H 6815 1346 50  0000 L CNN
-F 1 "0.1uF" H 6815 1255 50  0000 L CNN
+F 1 "100n" H 6815 1255 50  0000 L CNN
 F 2 "Capacitor_SMD:C_0603_1608Metric" H 6738 1150 50  0001 C CNN
 F 3 "" H 6700 1300 50  0001 C CNN
+F 4 "C1590" H 6700 1300 50  0001 C CNN "LCSC PN"
 	1    6700 1300
 	1    0    0    -1
@@
 P 7100 1300
 F 0 "C13" H 7215 1346 50  0000 L CNN
-F 1 "0.1uF" H 7215 1255 50  0000 L CNN
+F 1 "100n" H 7215 1255 50  0000 L CNN
 F 2 "Capacitor_SMD:C_0603_1608Metric" H 7138 1150 50  0001 C CNN
 F 3 "" H 7100 1300 50  0001 C CNN
+F 4 "C1590" H 7100 1300 50  0001 C CNN "LCSC PN"
 	1    7100 1300
 	1    0    0    -1
@@
 P 7500 1300
 F 0 "C14" H 7615 1346 50  0000 L CNN
-F 1 "0.1uF" H 7615 1255 50  0000 L CNN
+F 1 "100n" H 7615 1255 50  0000 L CNN
 F 2 "Capacitor_SMD:C_0603_1608Metric" H 7538 1150 50  0001 C CNN
 F 3 "" H 7500 1300 50  0001 C CNN
+F 4 "C1590" H 7500 1300 50  0001 C CNN "LCSC PN"
 	1    7500 1300
 	1    0    0    -1
@@
 P 7900 1300
 F 0 "C15" H 8015 1346 50  0000 L CNN
-F 1 "0.1uF" H 8015 1255 50  0000 L CNN
+F 1 "100n" H 8015 1255 50  0000 L CNN
 F 2 "Capacitor_SMD:C_0603_1608Metric" H 7938 1150 50  0001 C CNN
 F 3 "" H 7900 1300 50  0001 C CNN
+F 4 "C1590" H 7900 1300 50  0001 C CNN "LCSC PN"
 	1    7900 1300
 	1    0    0    -1
@@
 P 8300 1300
 F 0 "C16" H 8415 1346 50  0000 L CNN
-F 1 "0.1uF" H 8415 1255 50  0000 L CNN
+F 1 "100n" H 8415 1255 50  0000 L CNN
 F 2 "Capacitor_SMD:C_0603_1608Metric" H 8338 1150 50  0001 C CNN
 F 3 "" H 8300 1300 50  0001 C CNN
+F 4 "C1590" H 8300 1300 50  0001 C CNN "LCSC PN"
 	1    8300 1300
 	1    0    0    -1
@@
 P 8700 1300
 F 0 "C17" H 8815 1346 50  0000 L CNN
-F 1 "0.1uF" H 8815 1255 50  0000 L CNN
+F 1 "100n" H 8815 1255 50  0000 L CNN
 F 2 "Capacitor_SMD:C_0603_1608Metric" H 8738 1150 50  0001 C CNN
 F 3 "" H 8700 1300 50  0001 C CNN
+F 4 "C1590" H 8700 1300 50  0001 C CNN "LCSC PN"
 	1    8700 1300
 	1    0    0    -1
@@
 P 9100 1300
 F 0 "C18" H 9215 1346 50  0000 L CNN
-F 1 "0.1uF" H 9215 1255 50  0000 L CNN
+F 1 "100n" H 9215 1255 50  0000 L CNN
 F 2 "Capacitor_SMD:C_0603_1608Metric" H 9138 1150 50  0001 C CNN
 F 3 "" H 9100 1300 50  0001 C CNN
+F 4 "C1590" H 9100 1300 50  0001 C CNN "LCSC PN"
 	1    9100 1300
 	1    0    0    -1
@@
 P 9500 1300
 F 0 "C19" H 9615 1346 50  0000 L CNN
-F 1 "0.1uF" H 9615 1255 50  0000 L CNN
+F 1 "100n" H 9615 1255 50  0000 L CNN
 F 2 "Capacitor_SMD:C_0603_1608Metric" H 9538 1150 50  0001 C CNN
 F 3 "" H 9500 1300 50  0001 C CNN
+F 4 "C1590" H 9500 1300 50  0001 C CNN "LCSC PN"
 	1    9500 1300
 	1    0    0    -1
@@
 P 6700 2000
 F 0 "C20" H 6815 2046 50  0000 L CNN
-F 1 "0.1uF" H 6815 1955 50  0000 L CNN
+F 1 "100n" H 6815 1955 50  0000 L CNN
 F 2 "Capacitor_SMD:C_0603_1608Metric" H 6738 1850 50  0001 C CNN
 F 3 "" H 6700 2000 50  0001 C CNN
+F 4 "C1590" H 6700 2000 50  0001 C CNN "LCSC PN"
 	1    6700 2000
 	1    0    0    -1
@@
 P 7100 2000
 F 0 "C21" H 7215 2046 50  0000 L CNN
-F 1 "0.1uF" H 7215 1955 50  0000 L CNN
+F 1 "100n" H 7215 1955 50  0000 L CNN
 F 2 "Capacitor_SMD:C_0603_1608Metric" H 7138 1850 50  0001 C CNN
 F 3 "" H 7100 2000 50  0001 C CNN
+F 4 "C1590" H 7100 2000 50  0001 C CNN "LCSC PN"
 	1    7100 2000
 	1    0    0    -1
@@
 P 7500 2000
 F 0 "C22" H 7615 2046 50  0000 L CNN
-F 1 "0.1uF" H 7615 1955 50  0000 L CNN
+F 1 "100n" H 7615 1955 50  0000 L CNN
 F 2 "Capacitor_SMD:C_0603_1608Metric" H 7538 1850 50  0001 C CNN
 F 3 "" H 7500 2000 50  0001 C CNN
+F 4 "C1590" H 7500 2000 50  0001 C CNN "LCSC PN"
 	1    7500 2000
 	1    0    0    -1
@@
 P 7900 2000
 F 0 "C23" H 8015 2046 50  0000 L CNN
-F 1 "0.1uF" H 8015 1955 50  0000 L CNN
+F 1 "100n" H 8015 1955 50  0000 L CNN
 F 2 "Capacitor_SMD:C_0603_1608Metric" H 7938 1850 50  0001 C CNN
 F 3 "" H 7900 2000 50  0001 C CNN
+F 4 "C1590" H 7900 2000 50  0001 C CNN "LCSC PN"
 	1    7900 2000
 	1    0    0    -1
@@
 P 8300 2000
 F 0 "C24" H 8415 2046 50  0000 L CNN
-F 1 "0.1uF" H 8415 1955 50  0000 L CNN
+F 1 "100n" H 8415 1955 50  0000 L CNN
 F 2 "Capacitor_SMD:C_0603_1608Metric" H 8338 1850 50  0001 C CNN
 F 3 "" H 8300 2000 50  0001 C CNN
+F 4 "C1590" H 8300 2000 50  0001 C CNN "LCSC PN"
 	1    8300 2000
 	1    0    0    -1
@@
 P 8700 2000
 F 0 "C25" H 8815 2046 50  0000 L CNN
-F 1 "0.1uF" H 8815 1955 50  0000 L CNN
+F 1 "100n" H 8815 1955 50  0000 L CNN
 F 2 "Capacitor_SMD:C_0603_1608Metric" H 8738 1850 50  0001 C CNN
 F 3 "" H 8700 2000 50  0001 C CNN
+F 4 "C1590" H 8700 2000 50  0001 C CNN "LCSC PN"
 	1    8700 2000
 	1    0    0    -1
@@
 P 9100 2000
 F 0 "C26" H 9215 2046 50  0000 L CNN
-F 1 "0.1uF" H 9215 1955 50  0000 L CNN
+F 1 "100n" H 9215 1955 50  0000 L CNN
 F 2 "Capacitor_SMD:C_0603_1608Metric" H 9138 1850 50  0001 C CNN
 F 3 "" H 9100 2000 50  0001 C CNN
+F 4 "C1590" H 9100 2000 50  0001 C CNN "LCSC PN"
 	1    9100 2000
 	1    0    0    -1
@@
 P 9500 2000
 F 0 "C27" H 9615 2046 50  0000 L CNN
-F 1 "0.1uF" H 9615 1955 50  0000 L CNN
+F 1 "100n" H 9615 1955 50  0000 L CNN
 F 2 "Capacitor_SMD:C_0603_1608Metric" H 9538 1850 50  0001 C CNN
 F 3 "" H 9500 2000 50  0001 C CNN
+F 4 "C1590" H 9500 2000 50  0001 C CNN "LCSC PN"
 	1    9500 2000
 	1    0    0    -1

Commit message: Update: Add missing LCSC part numbers
Parts:
- RGB1, RGB10, RGB11, RGB12, RGB13, RGB14, RGB15, RGB16, RGB2, RGB3, RGB4, RGB5, RGB6, RGB7, RGB8, RGB9: LCSC PN (none) -> C114585
- U4: LCSC PN (none) -> C100024
Changed lines of the file:
@@
 F 2 "LED_SMD:LED_WS2812B_PLCC4_5.0x5.0mm_P3.2mm" H 2250 900 50  0001 L TNN
 F 3 "https://cdn-shop.adafruit.com/datasheets/WS2812B.pdf" H 2300 825 50  0001 L TNN
+F 4 "C114585" H 2200 1200 50  0001 C CNN "LCSC PN"
 	1    2200 1200
 	1    0    0    -1
@@
 F 2 "LED_SMD:LED_WS2812B_PLCC4_5.0x5.0mm_P3.2mm" H 2250 2000 50  0001 L TNN
 F 3 "https://cdn-shop.adafruit.com/datasheets/WS2812B.pdf" H 2300 1925 50  0001 L TNN
+F 4 "C114585" H 2200 2300 50  0001 C CNN "LCSC PN"
 	1    2200 2300
 	1    0    0    -1
@@
 F 2 "LED_SMD:LED_WS2812B_PLCC4_5.0x5.0mm_P3.2mm" H 2250 3200 50  0001 L TNN
 F 3 "https://cdn-shop.adafruit.com/datasheets/WS2812B.pdf" H 2300 3125 50  0001 L TNN
+F 4 "C114585" H 2200 3500 50  0001 C CNN "LCSC PN"
 	1    2200 3500
 	1    0    0    -1
@@
 F 2 "LED_SMD:LED_WS2812B_PLCC4_5.0x5.0mm_P3.2mm" H 2250 4300 50  0001 L TNN
 F 3 "https://cdn-shop.adafruit.com/datasheets/WS2812B.pdf" H 2300 4225 50  0001 L TNN
+F 4 "C114585" H 2200 4600 50  0001 C CNN "LCSC PN"
 	1    2200 4600
 	1    0    0    -1
@@
 F 2 "LED_SMD:LED_WS2812B_PLCC4_5.0x5.0mm_P3.2mm" H 2250 5400 50  0001 L TNN
 F 3 "https://cdn-shop.adafruit.com/datasheets/WS2812B.pdf" H 2300 5325 50  0001 L TNN
+F 4 "C114585" H 2200 5700 50  0001 C CNN "LCSC PN"
 	1    2200 5700
 	1    0    0    -1
@@
 F 2 "LED_SMD:LED_WS2812B_PLCC4_5.0x5.0mm_P3.2mm" H 2250 6400 50  0001 L TNN
 F 3 "https://cdn-shop.adafruit.com/datasheets/WS2812B.pdf" H 2300 6325 50  0001 L TNN
+F 4 "C114585" H 2200 6700 50  0001 C CNN "LCSC PN"
 	1    2200 6700
 	1    0    0    -1
@@
 F 2 "LED_SMD:LED_WS2812B_PLCC4_5.0x5.0mm_P3.2mm" H 3750 900 50  0001 L TNN
 F 3 "https://cdn-shop.adafruit.com/datasheets/WS2812B.pdf" H 3800 825 50  0001 L TNN
+F 4 "C114585" H 3700 1200 50  0001 C CNN "LCSC PN"
 	1    3700 1200
 	1    0    0    -1
@@
 F 2 "LED_SMD:LED_WS2812B_PLCC4_5.0x5.0mm_P3.2mm" H 3750 2000 50  0001 L TNN
 F 3 "https://cdn-shop.adafruit.com/datasheets/WS2812B.pdf" H 3800 1925 50  0001 L TNN
+F 4 "C114585" H 3700 2300 50  0001 C CNN "LCSC PN"
 	1    3700 2300
 	1    0    0    -1
@@
 F 2 "LED_SMD:LED_WS2812B_PLCC4_5.0x5.0mm_P3.2mm" H 3750 3200 50  0001 L TNN
 F 3 "https://cdn-shop.adafruit.com/datasheets/WS2812B.pdf" H 3800 3125 50  0001 L TNN
+F 4 "C114585" H 3700 3500 50  0001 C CNN "LCSC PN"
 	1    3700 3500
 	1    0    0    -1
@@
 F 2 "LED_SMD:LED_WS2812B_PLCC4_5.0x5.0mm_P3.2mm" H 3750 4300 50  0001 L TNN
 F 3 "https://cdn-shop.adafruit.com/datasheets/WS2812B.pdf" H 3800 4225 50  0001 L TNN
+F 4 "C114585" H 3700 4600 50  0001 C CNN "LCSC PN"
 	1    3700 4600
 	1    0    0    -1
@@
 F 2 "LED_SMD:LED_WS2812B_PLCC4_5.0x5.0mm_P3.2mm" H 3750 5400 50  0001 L TNN
 F 3 "https://cdn-shop.adafruit.com/datasheets/WS2812B.pdf" H 3800 5325 50  0001 L TNN
+F 4 "C114585" H 3700 5700 50  0001 C CNN "LCSC PN"
 	1    3700 5700
 	1    0    0    -1
@@
 F 2 "LED_SMD:LED_WS2812B_PLCC4_5.0x5.0mm_P3.2mm" H 3750 6400 50  0001 L TNN
 F 3 "https://cdn-shop.adafruit.com/datasheets/WS2812B.pdf" H 3800 6325 50  0001 L TNN
+F 4 "C114585" H 3700 6700 50  0001 C CNN "LCSC PN"
 	1    3700 6700
 	1    0    0    -1
@@
 F 2 "LED_SMD:LED_WS2812B_PLCC4_5.0x5.0mm_P3.2mm" H 5150 900 50  0001 L TNN
 F 3 "https://cdn-shop.adafruit.com/datasheets/WS2812B.pdf" H 5200 825 50  0001 L TNN
+F 4 "C114585" H 5100 1200 50  0001 C CNN "LCSC PN"
 	1    5100 1200
 	1    0    0    -1
@@
 F 2 "LED_SMD:LED_WS2812B_PLCC4_5.0x5.0mm_P3.2mm" H 5150 2000 50  0001 L TNN
 F 3 "https://cdn-shop.adafruit.com/datasheets/WS2812B.pdf" H 5200 1925 50  0001 L TNN
+F 4 "C114585" H 5100 2300 50  0001 C CNN "LCSC PN"
 	1    5100 2300
 	1    0    0    -1
@@
 F 2 "LED_SMD:LED_WS2812B_PLCC4_5.0x5.0mm_P3.2mm" H 5150 3200 50  0001 L TNN
 F 3 "https://cdn-shop.adafruit.com/datasheets/WS2812B.pdf" H 5200 3125 50  0001 L TNN
+F 4 "C114585" H 5100 3500 50  0001 C CNN "LCSC PN"
 	1    5100 3500
 	1    0    0    -1
@@
 F 2 "LED_SMD:LED_WS2812B_PLCC4_5.0x5.0mm_P3.2mm" H 5150 4300 50  0001 L TNN
 F 3 "https://cdn-shop.adafruit.com/datasheets/WS2812B.pdf" H 5200 4225 50  0001 L TNN
+F 4 "C114585" H 5100 4600 50  0001 C CNN "LCSC PN"
 	1    5100 4600
 	1    0    0    -1
@@
 F 7 "296-37176-1-ND" H 8200 3300 50  0001 L BNN "Field7"
 F 8 "SN74LV1T34DBVR" H 8200 3300 50  0001 L BNN "Field8"
+F 9 "C100024" H 8200 3300 50  0001 C CNN "LCSC PN"
 	1    8200 3300
 	1    0    0    -1

Commit message: Update: Switch voltage level shifter to different component
The initial component is out of stock at LCSC, so I found something that
I believe is similar, but is more readily available.
Parts:
- removed U4: SN74LV1T34DBVR, SOT95P280X145-5N, symbol SN74LV1T34DBVR:SN74LV1T34DBVR
- added U4: 74LVC1G34, Package_TO_SOT_SMD:SOT-353_SC-70-5, symbol 74LVC1G34:74LVC1G34
Connections:
- net +5V: now also U4.5 (VCC)
- net GND: now also U4.3 (GND)
- net RGBLED_3V3: now also U4.2
- net at RC9.2: now also U4.4
Changed lines of the file:
@@
-$EndComp
-$Comp
-L SN74LV1T34DBVR:SN74LV1T34DBVR U4
-U 1 1 5C2DFC20
-P 8200 3300
-F 0 "U4" H 8200 3767 50  0000 C CNN
-F 1 "SN74LV1T34DBVR" H 8200 3676 50  0000 C CNN
-F 2 "SOT95P280X145-5N" H 8200 3300 50  0001 L BNN
-F 3 "Single Power Supply BUFFER Logic Level Shifter _no enable_ 5-SOT-23 -40 to 125" H 8200 3300 50  0001 L BNN
-F 4 "https://www.digikey.ca/product-detail/en/texas-instruments/SN74LV1T34DBVR/296-37176-1-ND/4555593?utm_source=snapeda&utm_medium=aggregator&utm_campaign=symbol" H 8200 3300 50  0001 L BNN "Field4"
-F 5 "Texas Instruments" H 8200 3300 50  0001 L BNN "Field5"
-F 6 "SOT-23 Texas Instruments" H 8200 3300 50  0001 L BNN "Field6"
-F 7 "296-37176-1-ND" H 8200 3300 50  0001 L BNN "Field7"
-F 8 "SN74LV1T34DBVR" H 8200 3300 50  0001 L BNN "Field8"
-F 9 "C100024" H 8200 3300 50  0001 C CNN "LCSC PN"
-	1    8200 3300
-	1    0    0    -1
 $EndComp
 $Comp
 L power:+5V #PWR0158
 U 1 1 5C2E8AF6
-P 8725 2990
-F 0 "#PWR0158" H 8725 2840 50  0001 C CNN
-F 1 "+5V" H 8740 3163 50  0000 C CNN
-F 2 "" H 8725 2990 50  0001 C CNN
-F 3 "" H 8725 2990 50  0001 C CNN
-	1    8725 2990
+P 8150 3020
+F 0 "#PWR0158" H 8150 2870 50  0001 C CNN
+F 1 "+5V" H 8165 3193 50  0000 C CNN
+F 2 "" H 8150 3020 50  0001 C CNN
+F 3 "" H 8150 3020 50  0001 C CNN
+	1    8150 3020
 	1    0    0    -1
 $EndComp
-Wire Wire Line
-	8600 3100 8725 3100
-Wire Wire Line
-	8725 3100 8725 2990
 $Comp
 L power:GND #PWR0159
 U 1 1 5C2EB3B4
-P 8720 3650
-F 0 "#PWR0159" H 8720 3400 50  0001 C CNN
-F 1 "GND" H 8725 3477 50  0000 C CNN
-F 2 "" H 8720 3650 50  0001 C CNN
-F 3 "" H 8720 3650 50  0001 C CNN
-	1    8720 3650
+P 8150 3590
+F 0 "#PWR0159" H 8150 3340 50  0001 C CNN
+F 1 "GND" H 8155 3417 50  0000 C CNN
+F 2 "" H 8150 3590 50  0001 C CNN
+F 3 "" H 8150 3590 50  0001 C CNN
+	1    8150 3590
 	1    0    0    -1
 $EndComp
-Wire Wire Line
-	8600 3500 8720 3500
-Wire Wire Line
-	8720 3500 8720 3650
 Text GLabel 9235 3300 2    50   Input ~ 0
 RGBLED
 Text GLabel 7640 3300 0    50   Input ~ 0
 RGBLED_3V3
-Wire Wire Line
-	7640 3300 7800 3300
 Text GLabel 1750 1200 0    50   Input ~ 0
 RGBLED
@@
 $EndComp
 Wire Wire Line
-	8600 3300 8765 3300
+	9065 3300 9235 3300
+$Comp
+L 74LVC1G34:74LVC1G34 U4
+U 1 1 5C3F151C
+P 8200 3300
+F 0 "U4" H 8270 3410 50  0000 L CNN
+F 1 "74LVC1G34" H 8225 3180 50  0000 L CNN
+F 2 "Package_TO_SOT_SMD:SOT-353_SC-70-5" H 8200 3300 50  0001 C CNN
+F 3 "" H 8200 3300 50  0001 C CNN
+F 4 "C94111" H 8200 3300 50  0001 C CNN "LCSC PN"
+	1    8200 3300
+	1    0    0    -1
+$EndComp
 Wire Wire Line
-	9065 3300 9235 3300
+	7640 3300 7750 3300
+Wire Wire Line
+	8650 3300 8765 3300
+Wire Wire Line
+	8150 3020 8150 3100
+Wire Wire Line
+	8150 3590 8150 3500
 $EndSCHEMATC
